File: kicad/sensor-node-gamma.kicad_pcb (KiCad board)
At the start: 2 copper layers, 40 x 75 mm, 41 parts, among them SW1 SW_Push

Commit message: update PCB
Parts:
- removed REF** (x2): MountingHole_2.2mm_M2_Pad_Via, official stable:MountingHole_2.2mm_M2_Pad_Via
- removed RFM1: RFM98, sensor-node-gamma:RFM98
- removed the Ref** at (148.6, 110.0)
- removed the Ref** at (163.2, 133.1)
- removed the Ref** at (150.1, 118.0)
- removed the Ref** at (152.1, 114.5)
- removed the Ref** at (155.5, 104.8)
- removed the Ref** at (158.2, 101.8)
- removed the Ref** at (169.0, 103.5)
- removed the Ref** at (142.8, 122.0)
- removed the Ref** at (156.4, 121.2)
- removed the Ref** at (160.4, 120.9)
- removed the Ref** at (177.5, 114.2)
- removed the Ref** at (143.0, 111.5)
- removed the Ref** at (174.1, 97.3)
- removed the Ref** at (171.2, 110.7)
- removed the Ref** at (157.0, 112.0)
- removed the Ref** at (158.5, 107.8)
- removed the Ref** at (158.5, 109.8)
- removed the Ref** at (177.8, 126.8)
- removed the Ref** at (151.5, 127.8)
- removed the Ref** at (150.5, 131.4)
- added C10: 6.8pF, official stable:C_0402_1005Metric, F.Cu at (144.9, 98.4)
- added C11: 4.3pF, official stable:C_0402_1005Metric, F.Cu at (149.8, 99.7)
- added C12: 6.8pF, official stable:C_0402_1005Metric, F.Cu at (144.9, 101.4)
- added C13: 2.7pF, official stable:C_0402_1005Metric, F.Cu at (149.2, 103.2)
- added C14: 1.8pF, official stable:C_0402_1005Metric, F.Cu at (146.9, 102.9)
- added C15: 0.1µF, official stable:C_0603_1608Metric_Pad1.05x0.95mm_HandSolder, F.Cu at (147.5, 108.3)
- added C9: 270pF, official stable:C_0402_1005Metric, F.Cu at (146.9, 97.0)
- added L1: 18nH, official stable:L_0402_1005Metric, F.Cu at (146.9, 99.9)
- added L2: 56nH, official stable:L_0402_1005Metric, F.Cu at (148.8, 101.4)
- added L3: 16nH, official stable:L_0402_1005Metric, F.Cu at (151.9, 103.2)
- added L4: 16nH, official stable:L_0402_1005Metric, F.Cu at (147.8, 104.9)
- added L5: 220nH, official stable:L_0402_1005Metric, F.Cu at (150.5, 103.2)
- added Ref**: Val**, sensor-node-gamma:STICH, F.Cu at (169.9, 94.1)
- added Ref**: Val**, sensor-node-gamma:STICH, F.Cu at (149.9, 112.0)
- added Ref**: Val**, sensor-node-gamma:STICH, F.Cu at (164.8, 94.1)
- added Ref**: Val**, sensor-node-gamma:STICH, F.Cu at (159.7, 94.1)
- added Ref**: Val**, sensor-node-gamma:STICH, F.Cu at (154.6, 94.1)
- added Ref**: Val**, sensor-node-gamma:STICH, F.Cu at (166.9, 106.2)
- added Ref**: Val**, sensor-node-gamma:STICH, F.Cu at (169.2, 108.8)
- added Ref**: Val**, sensor-node-gamma:STICH, F.Cu at (165.4, 109.8)
- added Ref**: Val**, sensor-node-gamma:STICH, F.Cu at (157.6, 112.2)
- added Ref**: Val**, sensor-node-gamma:STICH, F.Cu at (152.6, 110.2)
- added S1: SHTC3, sensor-node-gamma:SHTC3, F.Cu at (152.6, 112.9)
- AE1: value Antenna -> Antenna_Chip; footprint sensor-node-gamma:ANT1204F002R0433A -> sensor-node-gamma:ANT-433-SP
- C1: value 0.1µF -> 1µF
- SI1: value Si7006 -> SI4012; footprint sensor-node-gamma:Si7006 -> official stable:MSOP-10_3x3mm_P0.5mm
- moved R2 24.7 mm to (157.3, 105.0), turned to 270 degrees
- moved R3 20.0 mm to (160.2, 106.0)
- moved R1 18.4 mm to (168.5, 116.6), turned to 90 degrees
- moved C2 17.4 mm to (174.6, 109.3)
- moved C3 17.4 mm to (174.6, 105.3)
- moved C4 17.4 mm to (174.6, 107.3)
- moved C5 17.4 mm to (174.6, 111.3)
- moved C6 17.3 mm to (160.6, 103.2)
- moved C7 17.3 mm to (160.6, 101.2)
- moved STM1 17.1 mm to (166.5, 108.2)
- moved SI1 15.8 mm to (152.9, 106.9), turned to 0 degrees
- moved C1 12.1 mm to (147.5, 110.5), turned to 0 degrees
- moved C8 8.82 mm to (152.6, 115.4), turned to 180 degrees
- moved AE1 7.26 mm to (159.6, 94.1), turned to 0 degrees
- moved G*** 0.71 mm to (160.5, 88.0)
Connections:
- C1 pad 1: /3V3 -> GND
- C1 pad 2: GND -> /3V3
- CD1 pad 6: (no net) -> Net-(CD1-Pad6)
- CD1 pad 7: (no net) -> Net-(CD1-Pad7)
- CD1 pad 8: (no net) -> Net-(CD1-Pad8)
- SI1 pad 1: /I2C_SDA -> Net-(SI1-Pad1)
- SI1 pad 3: (no net) -> Net-(C11-Pad1)
- SI1 pad 4: (no net) -> Net-(C14-Pad1)
- SI1 pad 6: /I2C_SCL -> Net-(SI1-Pad6)
- STM1 pad 10: /RFM_DIO1 -> Net-(STM1-Pad10)
- STM1 pad 11: /RFM_DIO0 -> Net-(STM1-Pad11)
- STM1 pad 12: /RFM_DIO4 -> Net-(STM1-Pad12)
- STM1 pad 13: /RFM_DIO3 -> Net-(STM1-Pad13)
- STM1 pad 14: /RFM_DIO5 -> Net-(STM1-Pad14)
- STM1 pad 15: (no net) -> Net-(STM1-Pad15)
- STM1 pad 18: (no net) -> Net-(STM1-Pad18)
- STM1 pad 2: (no net) -> Net-(STM1-Pad2)
- STM1 pad 21: (no net) -> /RFM_ENABLE
- STM1 pad 22: (no net) -> /~RFM_IRQ
- STM1 pad 25: /SPI_NSS -> Net-(STM1-Pad25)
- STM1 pad 26: /SPI_SCK -> Net-(STM1-Pad26)
- STM1 pad 27: /SPI_MISO -> Net-(STM1-Pad27)
- STM1 pad 28: /SPI_MOSI -> Net-(STM1-Pad28)
- STM1 pad 29: /RFM_RESET -> Net-(STM1-Pad29)
- STM1 pad 3: (no net) -> Net-(STM1-Pad3)
- STM1 pad 30: (no net) -> Net-(STM1-Pad30)
- STM1 pad 6: (no net) -> Net-(STM1-Pad6)
- STM1 pad 7: (no net) -> Net-(STM1-Pad7)
- STM1 pad 8: (no net) -> Net-(STM1-Pad8)
- STM1 pad 9: /RFM_DIO2 -> Net-(STM1-Pad9)
Routing:
- net /SPI_NSS: track 44.9 -> 0.00 mm, vias 2 -> 0
- net /SPI_SCK: track 41.8 -> 0.00 mm, vias 2 -> 0
- net /RFM_RESET: track 39.4 -> 0.00 mm
- net /SPI_MOSI: track 37.0 -> 0.00 mm
- net /RFM_DIO5: track 36.8 -> 0.00 mm
- net /SPI_MISO: track 35.1 -> 0.00 mm
- net /RFM_DIO3: track 20.3 -> 0.00 mm
- net GND: track 16.9 -> 35.9 mm, vias 0 -> 2
- net /RFM_DIO4: track 18.8 -> 0.00 mm
- net /3V3: track 120.5 -> 105.9 mm, vias 4 -> 2
- net /RFM_DIO0: track 12.5 -> 0.00 mm
- net Net-(C11-Pad1): track 0.00 -> 11.3 mm
- net /~SWD_RST: track 52.1 -> 40.9 mm, vias 2 -> 0
- net /RFM_DIO1: track 11.0 -> 0.00 mm
- net /RFM_DIO2: track 9.47 -> 0.00 mm
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Other:
- net class Default: trace_width 0.1 -> 0.25
- net class Limit added: clearance 0.1, trace_width 0.1, via_dia 0.45, via_drill 0.2
- board text added: "hochreiner.net sensor-node-gamma V1.1.0"
- board text removed: "hochreiner.net sensor-node-gamma V1.0.0"

Commit message: updated PCB
Parts:
- added REF**: MountingHole_2.2mm_M2_Pad_Via, official stable:MountingHole_2.2mm_M2_Pad_Via, F.Cu at (176.0, 139.0)
- added REF**: MountingHole_2.2mm_M2_Pad_Via, official stable:MountingHole_2.2mm_M2_Pad_Via, F.Cu at (144.0, 117.0)
- added Ref**: Val**, sensor-node-gamma:STICH, F.Cu at (166.5, 115.1)
- moved CD1 12.0 mm to (175.4, 129.4)
- moved BT1 11.0 mm to (169.5, 132.2)
- moved SW1 8.60 mm to (175.8, 118.2)
- moved C8 0.75 mm to (152.6, 116.2)
Routing:
- net /SWD_CLK: track 36.0 -> 24.4 mm
- net /SWD_IO: track 35.6 -> 24.1 mm
- net /~SWD_RST: track 40.9 -> 30.4 mm
- net /3V3: track 105.9 -> 97.0 mm
Other:
- board size 40 x 75 mm -> 40 x 63 mm
