File: kicad/sensor-node-gamma.kicad_pcb (KiCad board)
At the start: 2 copper layers, 40 x 75 mm, 27 parts, among them SW1 SW_Push

Commit message: changes antenna footprint
Parts:
- AE1: footprint sensor-node-gamma:ANT1204F002R0433A -> ANT1204F002R0433A
Routing:
- net Net-(AE1-Pad1): track 3.15 -> 4.65 mm
Changed lines of the file:
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@@
     (add_net "Net-(R1-Pad2)")
+  )
+  (module ANT1204F002R0433A (layer F.Cu)
+    (at 160 86.85 90)
+    (fp_text reference AE1 (at 3.85 3.1 90) (layer F.SilkS)
+      (effects (font (size 1 1) (thickness 0.15)))
+    )
+    (fp_text value Antenna (at 0 -3.35 90) (layer F.Fab)
+      (effects (font (size 1 1) (thickness 0.15)))
+    )
+    (fp_line (start -6.5 2) (end -6.5 -2) (layer F.Fab) (width 0.15))
+    (fp_line (start -8 2) (end -6.5 2) (layer F.Fab) (width 0.15))
+    (fp_line (start -8 -2) (end -8 2) (layer F.Fab) (width 0.15))
+    (fp_line (start -6.5 -2) (end -8 -2) (layer F.Fab) (width 0.15))
+    (fp_line (start -6.15 2) (end -6.15 -2) (layer F.SilkS) (width 0.15))
+    (fp_line (start 6.15 2) (end -6.15 2) (layer F.SilkS) (width 0.15))
+    (fp_line (start 6.15 -2) (end 6.15 2) (layer F.SilkS) (width 0.15))
+    (fp_line (start -6.15 -2) (end 6.15 -2) (layer F.SilkS) (width 0.15))
+    (pad "" smd rect (at 5.85 0 90) (size 1.3 4.5) (layers F.Cu F.Paste F.Mask))
+    (pad 1 smd rect (at -6.5 0 90) (size 1.3 4.5) (drill (offset 0.65 0)) (layers F.Cu F.Paste F.Mask)
+      (net 1 "Net-(AE1-Pad1)"))
   )
   (module sensor-node-gamma:STICH (layer F.Cu)
@@
     (pad 1 thru_hole circle (at 0 0) (size 0.6 0.6) (drill 0.3) (layers *.Cu)
       (net 3 GND) (zone_connect 2))
-  )
-  (module sensor-node-gamma:ANT1204F002R0433A (layer F.Cu)
-    (at 160 86.85 90)
-    (fp_text reference AE1 (at 3.85 3.1 90) (layer F.SilkS)
-      (effects (font (size 1 1) (thickness 0.15)))
-    )
-    (fp_text value Antenna (at 0 -3.35 90) (layer F.Fab)
-      (effects (font (size 1 1) (thickness 0.15)))
-    )
-    (fp_line (start -6.15 2) (end -6.15 -2) (layer F.SilkS) (width 0.15))
-    (fp_line (start 6.15 2) (end -6.15 2) (layer F.SilkS) (width 0.15))
-    (fp_line (start 6.15 -2) (end 6.15 2) (layer F.SilkS) (width 0.15))
-    (fp_line (start -6.15 -2) (end 6.15 -2) (layer F.SilkS) (width 0.15))
-    (pad "" smd rect (at 5.85 0 90) (size 1.3 4.5) (layers F.Cu F.Paste F.Mask))
-    (pad "" smd rect (at -5.85 0 90) (size 1.3 4.5) (layers F.Cu F.Paste F.Mask))
-    (pad 1 smd rect (at -8 0 90) (size 2 1.3) (drill (offset 1 0)) (layers F.Cu F.Paste F.Mask)
-      (net 1 "Net-(AE1-Pad1)"))
   )
   (module sensor-node-gamma:HU2032-LF (layer F.Cu)
@@
   (gr_line (start 180 80) (end 180 155) (layer Edge.Cuts) (width 0.15))
   (gr_line (start 140 80) (end 180 80) (layer Edge.Cuts) (width 0.15))
-  (segment (start 160 98) (end 160 94.85) (width 1.3) (layer F.Cu) (net 1))
+  (segment (start 160 98) (end 160 93.35) (width 1.2) (layer F.Cu) (net 1))
   (segment (start 171.04 143.5) (end 170.5 143.5) (width 0.25) (layer F.Cu) (net 2))
   (segment (start 170.5 143.5) (end 169.5 144.5) (width 0.25) (layer F.Cu) (net 2))

Commit message: updated to kicad 5
Parts:
- removed the Ref** at (178.5, 113.0)
- removed the Ref** at (160.0, 120.0)
- removed the Ref** at (172.0, 145.0)
- removed the Ref** at (160.5, 112.0)
- removed the Ref** at (163.0, 123.0)
- removed the Ref** at (157.0, 122.0)
- removed the Ref** at (160.7, 107.2)
- removed the Ref** at (167.1, 120.5)
- removed the Ref** at (173.4, 111.6)
- removed the Ref** at (153.9, 119.7)
- added Ref**: Val**, sensor-node-gamma:STICH, F.Cu at (178.6, 114.8)
- added Ref**: Val**, sensor-node-gamma:STICH, F.Cu at (166.0, 126.4)
- added Ref**: Val**, sensor-node-gamma:STICH, F.Cu at (163.2, 123.0)
- added Ref**: Val**, sensor-node-gamma:STICH, F.Cu at (173.2, 113.8)
- added Ref**: Val**, sensor-node-gamma:STICH, F.Cu at (160.4, 119.6)
- added Ref**: Val**, sensor-node-gamma:STICH, F.Cu at (161.6, 114.2)
- AE1: footprint ANT1204F002R0433A -> sensor-node-gamma:ANT1204F002R0433A
- C1, C2, C3, C4, C5, C6, C7: footprint Capacitors_SMD:C_0603_HandSoldering -> official stable:C_0603_1608Metric_Pad1.05x0.95mm_HandSolder
- R1, R2, R3: footprint Resistors_SMD:R_0603_HandSoldering -> official stable:R_0603_1608Metric_Pad1.05x0.95mm_HandSolder
- STM1: footprint Housings_QFP:LQFP-32_7x7mm_Pitch0.8mm -> official stable:LQFP-32_7x7mm_P0.8mm

Commit message: re-routed pcb
Parts:
- removed the Ref** at (178.6, 114.8)
- removed the Ref** at (166.0, 126.4)
- removed the Ref** at (163.2, 123.0)
- removed the Ref** at (173.2, 113.8)
- removed the Ref** at (160.4, 119.6)
- removed the Ref** at (161.6, 114.2)
- added REF**: MountingHole_2.2mm_M2_Pad_Via, official stable:MountingHole_2.2mm_M2_Pad_Via, F.Cu at (176.0, 151.0)
- added REF**: MountingHole_2.2mm_M2_Pad_Via, official stable:MountingHole_2.2mm_M2_Pad_Via, F.Cu at (144.0, 99.0)
- added Ref**: Val**, sensor-node-gamma:STICH, F.Cu at (177.8, 126.8)
- added Ref**: Val**, sensor-node-gamma:STICH, F.Cu at (142.8, 122.0)
- added Ref**: Val**, sensor-node-gamma:STICH, F.Cu at (156.4, 121.2)
- added Ref**: Val**, sensor-node-gamma:STICH, F.Cu at (160.4, 120.9)
- added Ref**: Val**, sensor-node-gamma:STICH, F.Cu at (177.5, 114.2)
- added Ref**: Val**, sensor-node-gamma:STICH, F.Cu at (174.1, 97.3)
- added Ref**: Val**, sensor-node-gamma:STICH, F.Cu at (151.5, 127.8)
- added Ref**: Val**, sensor-node-gamma:STICH, F.Cu at (150.5, 131.4)
- added Ref**: Val**, sensor-node-gamma:STICH, F.Cu at (163.2, 133.1)
- added Ref**: Val**, sensor-node-gamma:STICH, F.Cu at (150.1, 118.0)
- added Ref**: Val**, sensor-node-gamma:STICH, F.Cu at (152.1, 114.5)
- added Ref**: Val**, sensor-node-gamma:STICH, F.Cu at (155.5, 104.8)
- added Ref**: Val**, sensor-node-gamma:STICH, F.Cu at (158.2, 101.8)
- added Ref**: Val**, sensor-node-gamma:STICH, F.Cu at (169.0, 103.5)
- C7, R2, R3, SI1: moved to F.Cu
- moved C7 22.6 mm to (146.0, 109.0)
- moved R2 21.8 mm to (141.7, 124.1), turned to 90 degrees
- moved R1 21.2 mm to (154.6, 128.6), turned to 180 degrees
- moved C3 20.6 mm to (159.2, 113.4)
- moved C4 20.4 mm to (159.2, 115.4)
- moved C2 20.1 mm to (159.2, 117.4)
- moved STM1 19.9 mm to (151.6, 116.6)
- moved C5 19.9 mm to (159.2, 119.4)
- moved C6 18.6 mm to (145.0, 112.2), turned to 90 degrees
- moved SI1 18.4 mm to (142.7, 118.9), turned to 90 degrees
- moved RFM1 17.3 mm to (170.0, 103.8), turned to 180 degrees
- moved R3 16.6 mm to (141.7, 113.6), turned to 90 degrees
- moved C1 9.79 mm to (158.2, 104.8), turned to 180 degrees
- moved SW1 6.40 mm to (175.8, 126.8)
- moved CD1 4.14 mm to (175.4, 141.4)
Routing:
- net /SPI_NSS: track 16.2 -> 48.0 mm, vias 0 -> 2
- net /RFM_DIO2: track 33.9 -> 8.92 mm, vias 2 -> 0
- net /SPI_SCK: track 19.4 -> 43.7 mm, vias 0 -> 2
- net /RFM_RESET: track 17.4 -> 39.5 mm, vias 2 -> 0
- net /RFM_DIO1: track 29.5 -> 10.9 mm, vias 2 -> 0
- net /RFM_DIO5: track 18.3 -> 36.8 mm, vias 2 -> 0
- net /I2C_SCL: track 23.0 -> 8.91 mm, vias 1 -> 0
- net /RFM_DIO0: track 25.1 -> 12.5 mm, vias 2 -> 0
- net /SPI_MOSI: track 23.9 -> 36.1 mm
- net /SPI_MISO: track 26.2 -> 37.6 mm, vias 2 -> 0
- net /~SWD_RST: track 44.5 -> 53.4 mm, vias 0 -> 2
- net /I2C_SDA: track 19.1 -> 13.6 mm, vias 1 -> 0
- net Net-(R1-Pad2): track 2.57 -> 7.80 mm, vias 0 -> 2
- net /RFM_DIO3: track 15.3 -> 20.3 mm
- net GND: track 12.0 -> 7.30 mm, vias 1 -> 0
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
Commit message: re-rerouted pcb
Parts:
- added G***: LOGO, sensor-node-gamma:logo, B.Cu at (160.0, 87.5)
- added Ref**: Val**, sensor-node-gamma:STICH, F.Cu at (171.2, 110.7)
- added Ref**: Val**, sensor-node-gamma:STICH, F.Cu at (157.0, 112.0)
- added Ref**: Val**, sensor-node-gamma:STICH, F.Cu at (158.5, 107.8)
- added Ref**: Val**, sensor-node-gamma:STICH, F.Cu at (158.5, 109.8)
- moved C7 2.06 mm to (147.0, 110.8), turned to 90 degrees
Routing:
- net GND: track 7.30 -> 16.0 mm
- net /SPI_NSS: track 48.0 -> 44.9 mm
- net /3V3: track 116.2 -> 113.2 mm
- net /SPI_MISO: track 37.6 -> 35.1 mm
- net /SPI_SCK: track 43.7 -> 41.8 mm
- net /~SWD_RST: track 53.4 -> 52.1 mm
- net /SPI_MOSI: track 36.1 -> 37.0 mm
- net /RFM_DIO2: track 8.92 -> 9.47 mm
Other:
- outline, holes or cut-outs redrawn
- board text added: "sensor-node-gamma V1.0.0"

Commit message: added cap for sensor
Parts:
- added C8: 0.1µF, official stable:C_0603_1608Metric_Pad1.05x0.95mm_HandSolder, F.Cu at (143.8, 114.5)
- added Ref**: Val**, sensor-node-gamma:STICH, F.Cu at (148.6, 110.0)
- added Ref**: Val**, sensor-node-gamma:STICH, F.Cu at (143.0, 111.5)
- R2, R3: value R -> 10k
- moved C7 2.06 mm to (145.4, 109.5), turned to 180 degrees
- moved C6 0.87 mm to (145.4, 111.5), turned to 180 degrees
Routing:
- net /3V3: track 113.2 -> 120.5 mm
- net GND: track 16.0 -> 16.9 mm
Other:
- board text added: "hochreiner.net sensor-node-gamma V1.0.0"
- board text removed: "sensor-node-gamma V1.0.0"

Commit message: updated design rules and ran check
Other:
- net class Default: clearance 0.2 -> 0.1; trace_width 0.25 -> 0.1; via_dia 0.6 -> 0.45; via_drill 0.4 -> 0.2
- rule trace_clearance: 0.2 -> 0.1
- rule trace_min: 0.2 -> 0.1
- rule via_min_drill: 0.3 -> 0.2
- rule via_min_size: 0.4 -> 0.45
Changed lines of the file:
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@@
     (thickness 1.6)
     (drawings 9)
-    (tracks 186)
+    (tracks 185)
     (zones 0)
     (modules 41)
@@
   )
   (setup
-    (last_trace_width 0.25)
-    (trace_clearance 0.2)
+    (last_trace_width 0.1)
+    (trace_clearance 0.1)
     (zone_clearance 0.508)
     (zone_45_only no)
-    (trace_min 0.2)
+    (trace_min 0.1)
     (segment_width 0.2)
     (edge_width 0.15)
-    (via_size 0.6)
-    (via_drill 0.4)
-    (via_min_size 0.4)
-    (via_min_drill 0.3)
+    (via_size 0.45)
+    (via_drill 0.2)
+    (via_min_size 0.45)
+    (via_min_drill 0.2)
     (uvia_size 0.3)
     (uvia_drill 0.1)
@@
   (net 20 /RFM_DIO2)
   (net_class Default "This is the default net class."
-    (clearance 0.2)
-    (trace_width 0.25)
-    (via_dia 0.6)
-    (via_drill 0.4)
+    (clearance 0.1)
+    (trace_width 0.1)
+    (via_dia 0.45)
+    (via_drill 0.2)
     (uvia_dia 0.3)
     (uvia_drill 0.1)
@@
   (gr_line (start 180 82) (end 180 153) (layer Edge.Cuts) (width 0.15))
   (gr_line (start 142 80) (end 178 80) (layer Edge.Cuts) (width 0.15))
-  (segment (start 176 142.684998) (end 176 143) (width 0.25) (layer F.Cu) (net 0))
   (segment (start 161 96.8) (end 160 95.8) (width 1.2) (layer F.Cu) (net 1))
   (segment (start 160 95.8) (end 160 93.35) (width 1.2) (layer F.Cu) (net 1))

Commit message: completed hybrid version
Parts:
- removed the REF** at (176.0, 151.0)
- removed the REF** at (144.0, 99.0)
- removed Ref** (x20): Val**, sensor-node-gamma:STICH
- removed SI1: Si7006, sensor-node-gamma:Si7006
- added REF**: MountingHole_2.2mm_M2_Pad_Via, official stable:MountingHole_2.2mm_M2_Pad_Via, F.Cu at (144.0, 151.0)
- added REF**: MountingHole_2.2mm_M2_Pad_Via, official stable:MountingHole_2.2mm_M2_Pad_Via, F.Cu at (176.0, 99.0)
- added S1: SHTC3, sensor-node-gamma:SHTC3, F.Cu at (147.9, 134.5)
- moved SW1 30.8 mm to (154.3, 148.9)
- moved CD1 24.7 mm to (150.7, 140.3), turned to 90 degrees
- moved C7 23.3 mm to (157.3, 129.5), turned to 0 degrees
- moved R3 19.6 mm to (152.4, 129.9), turned to 0 degrees
- moved C8 17.4 mm to (147.9, 131.4), turned to 0 degrees
- moved RFM1 17.2 mm to (153.0, 106.1), turned to 90 degrees
- moved BT1 17.0 mm to (169.2, 126.2), turned to 270 degrees
- moved R2 14.2 mm to (153.3, 132.2), turned to 180 degrees
- moved C1 11.4 mm to (151.1, 95.9)
- moved C5 8.45 mm to (157.3, 127.7)
- moved C2 7.18 mm to (158.2, 124.5), turned to 270 degrees
- moved C3 6.35 mm to (159.0, 119.8)
- moved C4 6.30 mm to (158.9, 121.7)
- moved C6 6.26 mm to (145.8, 117.7)
- moved STM1 5.95 mm to (151.7, 122.5)
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Connections:
- STM1 pad 10: /RFM_DIO1 -> /SPI_NSS
- STM1 pad 11: /RFM_DIO0 -> /SPI_SCK
- STM1 pad 12: /RFM_DIO4 -> (no net)
- STM1 pad 13: /RFM_DIO3 -> /SPI_MOSI
- STM1 pad 14: /RFM_DIO5 -> /SPI_MISO
- STM1 pad 18: (no net) -> /RFM_DIO3
- STM1 pad 19: /I2C_SCL -> /RFM_DIO4
- STM1 pad 20: /I2C_SDA -> /RFM_DIO0
- STM1 pad 21: (no net) -> /RFM_DIO1
- STM1 pad 22: (no net) -> /RFM_DIO2
- STM1 pad 25: /SPI_NSS -> (no net)
- STM1 pad 26: /SPI_SCK -> (no net)
- STM1 pad 27: /SPI_MISO -> (no net)
- STM1 pad 28: /SPI_MOSI -> (no net)
- STM1 pad 29: /RFM_RESET -> /I2C_SCL
- STM1 pad 30: (no net) -> /I2C_SDA
- STM1 pad 8: (no net) -> /RFM_DIO5
- STM1 pad 9: /RFM_DIO2 -> /RFM_RESET
Routing:
- net /SPI_NSS: track 44.9 -> 4.82 mm, vias 2 -> 0
- net /SPI_SCK: track 41.8 -> 5.07 mm, vias 2 -> 0
- net /RFM_RESET: track 39.4 -> 5.32 mm
- net /SPI_MOSI: track 37.0 -> 5.24 mm
- net /RFM_DIO5: track 36.8 -> 7.00 mm
- net /SPI_MISO: track 35.1 -> 5.74 mm
- net /SWD_CLK: track 43.7 -> 18.3 mm
- net /SWD_IO: track 43.5 -> 18.7 mm
- net /3V3: track 120.5 -> 97.4 mm, vias 4 -> 6
- net /RFM_DIO2: track 9.47 -> 30.5 mm
- net /RFM_DIO1: track 11.0 -> 29.9 mm
- net /RFM_DIO0: track 12.5 -> 29.4 mm
- net /~SWD_RST: track 52.1 -> 36.3 mm, vias 2 -> 0
- net /RFM_DIO4: track 18.8 -> 29.7 mm
- net GND: track 16.9 -> 27.7 mm, vias 0 -> 37
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Other:
- net class Antenna added: clearance 0.15, trace_width 1.2, via_dia 0.45, via_drill 0.2
- net class Default: clearance 0.1 -> 0.15; trace_width 0.1 -> 0.2
- net class Power added: clearance 0.15, trace_width 0.3, via_dia 0.45, via_drill 0.2
- rule trace_clearance: 0.1 -> 0.15
- board text added: "hochreiner.net sensor-node-gamma hybrid - V1.0.0"
- board text removed: "hochreiner.net sensor-node-gamma V1.0.0"
